File: PCB/wled_esp_32_v1.kicad_pcb (KiCad board)
At the start: 2 copper layers, 23 parts, among them J1 PWR IN, J2 Neopixel_1, J3 PWM_STRIP_1, Q1 IRFR024N, Q2 IRFR024N, Q3 IRFR5305, Q4 MMBT2222A, U1 XIAO-ESP32-C3-SMD, U2 74AHCT244, U3 AMS1117-3.3

Commit message: checkpoint pcb files
Parts:
- removed C1, C2, C3: 0.1uf, Capacitor_SMD:C_1206_3216Metric_Pad1.33x1.80mm_HandSolder
- removed R1: R_Small, Resistor_SMD:R_1206_3216Metric_Pad1.30x1.75mm_HandSolder
- removed U3: AMS1117-3.3, Package_TO_SOT_SMD:SOT-223-3_TabPin2
- U1: footprint Seeed Studio XIAO Series Library:XIAO-ESP32C3-DIP -> Seeed Studio XIAO Series Library:XIAO-ESP32C3-SMD
- moved J2 80.5 mm to (93.5, 35.5), turned to 90 degrees
- moved J1 70.3 mm to (28.0, 31.9), turned to -90 degrees
- moved J3 51.0 mm to (93.5, 51.1), turned to 90 degrees
- moved Q3 45.0 mm to (74.7, 26.5)
- moved Q2 38.4 mm to (74.7, 50.0)
- moved Q1 38.0 mm to (74.7, 38.2)
- moved C5 33.2 mm to (58.1, 25.0), turned to -90 degrees
- moved U2 31.4 mm to (45.4, 50.0), turned to -90 degrees
- moved R8 28.2 mm to (61.6, 25.0), turned to -90 degrees
- moved Q4 27.2 mm to (62.5, 32.6), turned to 90 degrees
- moved C4 24.1 mm to (58.1, 46.5), turned to -90 degrees
- moved R6 21.6 mm to (65.1, 25.0), turned to -90 degrees
- moved R7 18.3 mm to (58.1, 32.5), turned to -90 degrees
- moved R3 16.4 mm to (64.5, 53.0), turned to 90 degrees
- moved R5 12.3 mm to (58.1, 54.0), turned to 90 degrees
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Connections:
- U1 pad 11: NEOPIXEL1_DATA_3V3 -> PWM1_DATA
- U1 pad 2: PWM1_DATA -> NEOPIXEL1_PWR_DPIN_3V3
- U1 pad 3: NEOPIXEL1_PWR_DPIN_3V3 -> NEOPIXEL1_DATA_3V3
