File: PCB/wled_esp_32_v1.kicad_sch (KiCad schematic)
At the start: 23 parts, among them J1 PWR IN, J2 Neopixel_1, J3 PWM_STRIP_1, Q1 IRFR024N, Q2 IRFR024N, Q3 IRFR5305, Q4 MMBT2222A, U1 XIAO-ESP32-C3-SMD, U2 74AHCT244, U3 AMS1117-3.3

Commit message: checkpoint pcb files
Parts:
- removed C1: 0.1uf, Capacitor_SMD:C_1206_3216Metric_Pad1.33x1.80mm_HandSolder, symbol Device:C_Small
- removed R1: R_Small, Resistor_SMD:R_1206_3216Metric_Pad1.30x1.75mm_HandSolder, symbol Device:R_Small
- U1: footprint Seeed Studio XIAO Series Library:XIAO-ESP32C3-DIP -> Seeed Studio XIAO Series Library:XIAO-ESP32C3-SMD
Connections:
- net NEOPIXEL1_DATA_3V3: now also U1.3 (GPIO4_A2_D2); no longer U1.11 (GPIO10_D10_MOSI)
- net NEOPIXEL1_PWR_DPIN_3V3: now also U1.2 (GPIO3_A1_D1); no longer U1.3 (GPIO4_A2_D2)
- net PWM1_DATA: now also U1.11 (GPIO10_D10_MOSI); no longer U1.2 (GPIO3_A1_D1)
Other:
- note added: "MCU - ESP32"
- note removed: "MCU - ESP33"
Changed lines of the file:
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@@
 	(generator_version "9.0")
 	(paper "A4")
-	(text "MCU - ESP33"
+	(text "MCU - ESP32\n"
 		(exclude_from_sim no)
 		(at 185.928 14.732 0)
@@
 		)
 	)
-	(global_label "PWM1_DATA"
+	(global_label "NEOPIXEL1_DATA_3V3"
 		(shape input)
-		(at 203.2 45.72 180)
+		(at 115.57 87.63 180)
 		(fields_autoplaced yes)
 		(effects
@@
 		)
 		(property "Intersheetrefs" "${INTERSHEET_REFS}"
-			(at 189.4501 45.72 0)
+			(at 92.4463 87.63 0)
 			(effects
 				(font
@@
 		)
 	)
-	(global_label "NEOPIXEL1_DATA_3V3"
+	(global_label "NEOPIXEL1_PWR_DPIN_3V3"
 		(shape input)
-		(at 115.57 87.63 180)
+		(at 203.2 45.72 180)
 		(fields_autoplaced yes)
 		(effects
@@
 		)
 		(property "Intersheetrefs" "${INTERSHEET_REFS}"
-			(at 92.4463 87.63 0)
+			(at 175.0568 45.72 0)
 			(effects
 				(font
@@
 	(global_label "NEOPIXEL1_DATA_3V3"
 		(shape input)
-		(at 257.81 53.34 0)
+		(at 204.47 49.53 180)
 		(fields_autoplaced yes)
 		(effects
@@
 				(size 1.27 1.27)
 			)
-			(justify left)
+			(justify right)
 		)
 		(property "Intersheetrefs" "${INTERSHEET_REFS}"
-			(at 280.9337 53.34 0)
+			(at 181.3463 49.53 0)
 			(effects
 				(font
 					(size 1.27 1.27)
 				)
-				(justify left)
+				(justify right)
 				(hide yes)
 			)
 		)
 	)
-	(global_label "NEOPIXEL1_PWR_DPIN_3V3"
+	(global_label "NEOPIXEL1_PWR_OUT"
 		(shape input)
-		(at 204.47 49.53 180)
+		(at 148.59 45.72 0)
 		(fields_autoplaced yes)
 		(effects
@@
 				(size 1.27 1.27)
 			)
-			(justify right)
+			(justify left)
 		)
 		(property "Intersheetrefs" "${INTERSHEET_REFS}"
-			(at 176.3268 49.53 0)
+			(at 171.4113 45.72 0)
 			(effects
 				(font
 					(size 1.27 1.27)
 				)
-				(justify right)
+				(justify left)
 				(hide yes)
 			)
 		)
 	)
-	(global_label "NEOPIXEL1_PWR_OUT"
+	(global_label "PWM1_DATA"
 		(shape input)
-		(at 148.59 45.72 0)
+		(at 257.81 53.34 0)
 		(fields_autoplaced yes)
 		(effects
@@
 		)
 		(property "Intersheetrefs" "${INTERSHEET_REFS}"
-			(at 171.4113 45.72 0)
+			(at 271.5599 53.34 0)
 			(effects
 				(font
@@
 		(exclude_from_sim no)
 		(in_bom yes)
-		(on_board yes)
+		(on_board no)
 		(dnp no)
 		(fields_autoplaced yes)
@@
 		(exclude_from_sim no)
 		(in_bom yes)
-		(on_board yes)
+		(on_board no)
 		(dnp no)
 		(fields_autoplaced yes)
@@
 		(exclude_from_sim no)
 		(in_bom yes)
-		(on_board yes)
+		(on_board no)
 		(dnp no)
 		(fields_autoplaced yes)
@@
 		(exclude_from_sim no)
 		(in_bom yes)
-		(on_board yes)
+		(on_board no)
 		(dnp no)
 		(fields_autoplaced yes)
@@
 		(exclude_from_sim no)
 		(in_bom yes)
-		(on_board yes)
+		(on_board no)
 		(dnp no)
 		(property "Reference" "#PWR02"
@@
 	)
 	(symbol
-		(lib_id "Device:R_Small")
-		(at 241.3 133.35 0)
-		(unit 1)
-		(exclude_from_sim no)
-		(in_bom yes)
-		(on_board yes)
-		(dnp no)
-		(fields_autoplaced yes)
-		(property "Reference" "R1"
-			(at 243.84 132.0799 0)
-			(effects
-				(font
-					(size 1.27 1.27)
-				)
-				(justify left)
-			)
-		)
-		(property "Value" "R_Small"
-			(at 243.84 134.6199 0)
-			(effects
-				(font
-					(size 1.27 1.27)
-				)
-				(justify left)
-			)
-		)
-		(property "Footprint" "Resistor_SMD:R_1206_3216Metric_Pad1.30x1.75mm_HandSolder"
-			(at 241.3 133.35 0)
-			(effects
-				(font
-					(size 1.27 1.27)
-				)
-				(hide yes)
-			)
-		)
-		(property "Datasheet" "~"
-			(at 241.3 133.35 0)
-			(effects
-				(font
-					(size 1.27 1.27)
-				)
-				(hide yes)
-			)
-		)
-		(property "Description" "Resistor, small symbol"
-			(at 241.3 133.35 0)
-			(effects
-				(font
-					(size 1.27 1.27)
-				)
-				(hide yes)
-			)
-		)
-		(pin "1"
-		)
-		(pin "2"
-		)
-		(instances
-			(project ""
-				(path "/d2d38338-08e5-4e30-a0a2-fb1dbe6e0d27"
-					(reference "R1")
-					(unit 1)
-				)
-			)
-		)
-	)
-	(symbol
 		(lib_id "power:+5V")
 		(at 132.08 74.93 0)
@@
 	(symbol
 		(lib_id "Device:C_Small")
-		(at 260.35 132.08 0)
-		(unit 1)
-		(exclude_from_sim no)
-		(in_bom yes)
-		(on_board yes)
-		(dnp no)
-		(fields_autoplaced yes)
-		(property "Reference" "C1"
-			(at 262.89 130.8162 0)
-			(effects
-				(font
-					(size 1.27 1.27)
-				)
-				(justify left)
-			)
-		)
-		(property "Value" "0.1uf"
-			(at 262.89 133.3562 0)
-			(effects
-				(font
-					(size 1.27 1.27)
-				)
-				(justify left)
-			)
-		)
-		(property "Footprint" "Capacitor_SMD:C_1206_3216Metric_Pad1.33x1.80mm_HandSolder"
-			(at 260.35 132.08 0)
-			(effects
-				(font
-					(size 1.27 1.27)
-				)
-				(hide yes)
-			)
-		)
-		(property "Datasheet" "~"
-			(at 260.35 132.08 0)
-			(effects
-				(font
-					(size 1.27 1.27)
-				)
-				(hide yes)
-			)
-		)
-		(property "Description" "Unpolarized capacitor, small symbol"
-			(at 260.35 132.08 0)
-			(effects
-				(font
-					(size 1.27 1.27)
-				)
-				(hide yes)
-			)
-		)
-		(pin "2"
-		)
-		(pin "1"
-		)
-		(instances
-			(project ""
-				(path "/d2d38338-08e5-4e30-a0a2-fb1dbe6e0d27"
-					(reference "C1")
-					(unit 1)
-				)
-			)
-		)
-	)
-	(symbol
-		(lib_id "Device:C_Small")
 		(at 146.05 120.65 90)
 		(unit 1)
@@
 			)
 		)
-		(property "Footprint" "Seeed Studio XIAO Series Library:XIAO-ESP32C3-DIP"
+		(property "Footprint" "Seeed Studio XIAO Series Library:XIAO-ESP32C3-SMD"
 			(at 223.52 48.26 0)
 			(effects
@@
 		(exclude_from_sim no)
 		(in_bom yes)
-		(on_board yes)
+		(on_board no)
 		(dnp no)
 		(fields_autoplaced yes)
